File: Hardware/io2db9.brd (EAGLE design)
At the start: 94.1 x 31.2 mm, 22 parts

Commit message: actualizo io2db9
Parts:
- moved J1 1.00 mm to (84.0, -4.38)
Routing:
- net 1PFIRE1: track 24.2 -> 25.2 mm
- net 1PDOWN: track 21.2 -> 21.9 mm
- net 1PUP: track 24.4 -> 25.0 mm
- net 1PLEFT: track 12.3 -> 12.9 mm
- net 1PMUX: track 45.3 -> 44.8 mm
Other:
- board size 94.1 x 31.2 mm -> 95.1 x 31.2 mm
