File: Hardware/db9nes.brd (EAGLE design)
At the start: 53.1 x 25.9 mm, 3 parts

Commit message: updated
Parts:
- added R1, R2, R3: 3k6, resistor:R0603
- moved U$1 5.33 mm to (38.9, 10.6)
Connections:
- net 5V: now also R1.1, R2.1, R3.1
- net CLK1: now also R1.2
- net CLK2: now also R3.2
- net LAT: now also R2.2
Routing:
- net 5V: track 36.0 -> 57.6 mm
- net CLK2: track 24.1 -> 38.3 mm
- net CLK1: track 4.50 -> 12.6 mm
- net LAT: track 36.8 -> 43.9 mm
- net GND: track 41.4 -> 46.8 mm
- net DAT2: track 24.3 -> 29.6 mm
- net D4_2: track 23.4 -> 28.7 mm
Other:
- board size 53.1 x 25.9 mm -> 58.4 x 25.9 mm
Changed lines of the file:
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@@
 <board>
 <plain>
-<wire x1="53.086" y1="25.908" x2="0" y2="25.908" width="0" layer="20"/>
+<wire x1="58.42" y1="25.908" x2="0" y2="25.908" width="0" layer="20"/>
 <hole x="23.20798125" y="2.34441875" drill="4.318"/>
 <hole x="3.141975" y="2.32918125" drill="4.318"/>
-<hole x="49.77638125" y="2.34441875" drill="4.318"/>
-<hole x="29.710375" y="2.32918125" drill="4.318"/>
-<wire x1="0" y1="0" x2="53.086" y2="0" width="0" layer="20"/>
-<wire x1="53.086" y1="0" x2="53.086" y2="25.908" width="0" layer="20"/>
+<hole x="55.11038125" y="2.34441875" drill="4.318"/>
+<hole x="35.044375" y="2.32918125" drill="4.318"/>
+<wire x1="0" y1="0" x2="58.42" y2="0" width="0" layer="20"/>
+<wire x1="58.42" y1="0" x2="58.42" y2="25.908" width="0" layer="20"/>
 <wire x1="0" y1="0" x2="0" y2="25.908" width="0" layer="20"/>
 </plain>
@@
 </element>
 <element name="U$2" library="gamepad-conn" package="NESCONN_NO_TABS" value="NESCONNNO_TABS" x="6.9596" y="10.5664"/>
-<element name="U$1" library="gamepad-conn" package="NESCONN_NO_TABS" value="NESCONNNO_TABS" x="33.528" y="10.5664"/>
+<element name="U$1" library="gamepad-conn" package="NESCONN_NO_TABS" value="NESCONNNO_TABS" x="38.862" y="10.5664"/>
+<element name="R1" library="resistor" library_urn="urn:adsk.eagle:library:348" package="R0603" package3d_urn="urn:adsk.eagle:package:26057/1" value="3k6" x="13.97" y="7.366" smashed="yes" rot="MR0"/>
+<element name="R2" library="resistor" library_urn="urn:adsk.eagle:library:348" package="R0603" package3d_urn="urn:adsk.eagle:package:26057/1" value="3k6" x="43.942" y="18.542" smashed="yes" rot="MR0"/>
+<element name="R3" library="resistor" library_urn="urn:adsk.eagle:library:348" package="R0603" package3d_urn="urn:adsk.eagle:package:26057/1" value="3k6" x="48.768" y="6.858" smashed="yes" rot="MR180"/>
 </elements>
 <signals>
 <signal name="GND">
 <polygon width="0.4064" layer="1">
-<vertex x="52.578" y="25.4"/>
-<vertex x="0.254" y="25.908"/>
+<vertex x="58.166" y="25.654"/>
+<vertex x="0.254" y="25.654"/>
 <vertex x="0.254" y="0.508"/>
-<vertex x="52.578" y="0.508"/>
+<vertex x="58.166" y="0.254"/>
 </polygon>
 <contactref element="J1" pad="8"/>
 <polygon width="0.4064" layer="16">
-<vertex x="52.578" y="25.654"/>
-<vertex x="0.254" y="25.908"/>
-<vertex x="0.254" y="0.508"/>
-<vertex x="52.578" y="0.508"/>
+<vertex x="58.166" y="25.654"/>
+<vertex x="0.254" y="25.654"/>
+<vertex x="0.254" y="0.254"/>
+<vertex x="58.166" y="0.254"/>
 </polygon>
 <contactref element="U$2" pad="GND"/>
@@
 <wire x1="20.32" y1="19.558" x2="20.32" y2="15.7988" width="0.254" layer="1"/>
 <contactref element="U$1" pad="GND"/>
-<wire x1="45.72" y1="14.6304" x2="36.7284" y2="23.622" width="0.254" layer="1"/>
-<wire x1="19.916" y1="23.622" x2="17.78" y2="21.486" width="0.254" layer="1"/>
-<wire x1="36.7284" y1="23.622" x2="19.916" y2="23.622" width="0.254" layer="1"/>
+<wire x1="17.78" y1="21.486" x2="19.916" y2="23.622" width="0.254" layer="1"/>
+<wire x1="42.0624" y1="23.622" x2="51.054" y2="14.6304" width="0.254" layer="1"/>
+<wire x1="19.916" y1="23.622" x2="42.0624" y2="23.622" width="0.254" layer="1"/>
 </signal>
 <signal name="5V">
@@
 <wire x1="21.796" y1="14.684" x2="17.6784" y2="10.5664" width="0.254" layer="1"/>
 <contactref element="U$1" pad="5V"/>
-<wire x1="41.656" y1="10.5664" x2="39.2176" y2="8.128" width="0.254" layer="1"/>
-<wire x1="28.4" y1="8.128" x2="21.796" y2="14.732" width="0.254" layer="1"/>
-<wire x1="39.2176" y1="8.128" x2="28.4" y2="8.128" width="0.254" layer="1"/>
+<wire x1="21.796" y1="14.732" x2="28.4" y2="8.128" width="0.254" layer="1"/>
+<contactref element="R1" pad="1"/>
+<contactref element="R2" pad="1"/>
+<contactref element="R3" pad="1"/>
+<wire x1="44.792" y1="18.542" x2="44.792" y2="12.7644" width="0.254" layer="16"/>
+<wire x1="44.792" y1="12.7644" x2="46.99" y2="10.5664" width="0.254" layer="16"/>
+<wire x1="44.5516" y1="8.128" x2="46.99" y2="10.5664" width="0.254" layer="1"/>
+<wire x1="28.4" y1="8.128" x2="44.5516" y2="8.128" width="0.254" layer="1"/>
+<wire x1="14.82" y1="7.366" x2="14.82" y2="10.2988" width="0.254" layer="16"/>
+<wire x1="14.82" y1="10.2988" x2="15.0876" y2="10.5664" width="0.254" layer="16"/>
+<wire x1="47.918" y1="6.858" x2="47.918" y2="9.6384" width="0.254" layer="16"/>
+<wire x1="47.918" y1="9.6384" x2="46.99" y2="10.5664" width="0.254" layer="16"/>
 </signal>
 <signal name="CLK1">
@@
 <wire x1="16.256" y1="18.646" x2="16.256" y2="15.7988" width="0.254" layer="1"/>
 <wire x1="16.256" y1="15.7988" x2="15.0876" y2="14.6304" width="0.254" layer="1"/>
+<contactref element="R1" pad="2"/>
+<wire x1="13.12" y1="7.366" x2="13.12" y2="12.6628" width="0.254" layer="16"/>
+<wire x1="13.12" y1="12.6628" x2="15.0876" y2="14.6304" width="0.254" layer="16"/>
 </signal>
 <signal name="DAT1">
@@
 <wire x1="12.192" y1="15.7988" x2="11.0236" y2="14.6304" width="0.254" layer="1"/>
 <wire x1="12.192" y1="19.558" x2="12.192" y2="15.7988" width="0.254" layer="1"/>
-<wire x1="14.876" y1="21.486" x2="16.758" y2="23.368" width="0.254" layer="16"/>
-<wire x1="37.592" y1="16.002" x2="37.592" y2="14.6304" width="0.254" layer="16"/>
-<wire x1="16.758" y1="23.368" x2="30.226" y2="23.368" width="0.254" layer="16"/>
-<wire x1="30.226" y1="23.368" x2="37.592" y2="16.002" width="0.254" layer="16"/>
+<wire x1="16.758" y1="23.368" x2="14.876" y2="21.486" width="0.254" layer="16"/>
+<contactref element="R2" pad="2"/>
+<wire x1="42.926" y1="14.6304" x2="42.926" y2="18.376" width="0.254" layer="16"/>
+<wire x1="42.926" y1="18.376" x2="43.092" y2="18.542" width="0.254" layer="16"/>
+<wire x1="43.092" y1="18.542" x2="38.266" y2="23.368" width="0.254" layer="16"/>
+<wire x1="38.266" y1="23.368" x2="16.758" y2="23.368" width="0.254" layer="16"/>
 </signal>
 <signal name="DAT2">
@@
 <contactref element="U$1" pad="D0"/>
 <wire x1="12.106" y1="21.486" x2="13.526" y2="20.066" width="0.254" layer="16"/>
-<wire x1="27.7876" y1="14.6304" x2="33.528" y2="14.6304" width="0.254" layer="16"/>
+<wire x1="27.7876" y1="14.6304" x2="38.862" y2="14.6304" width="0.254" layer="16"/>
 <wire x1="13.526" y1="20.066" x2="22.352" y2="20.066" width="0.254" layer="16"/>
 <wire x1="22.352" y1="20.066" x2="27.7876" y2="14.6304" width="0.254" layer="16"/>
@@
 <contactref element="U$1" pad="CLOCK"/>
 <wire x1="20.406" y1="21.486" x2="21.44" y2="21.486" width="0.254" layer="1"/>
-<wire x1="39.5224" y1="16.764" x2="41.656" y2="14.6304" width="0.254" layer="1"/>
 <wire x1="21.44" y1="21.486" x2="26.162" y2="16.764" width="0.254" layer="1"/>
-<wire x1="26.162" y1="16.764" x2="39.5224" y2="16.764" width="0.254" layer="1"/>
+<contactref element="R3" pad="2"/>
+<wire x1="44.8564" y1="16.764" x2="46.99" y2="14.6304" width="0.254" layer="1"/>
+<wire x1="26.162" y1="16.764" x2="44.8564" y2="16.764" width="0.254" layer="1"/>
+<wire x1="49.618" y1="6.858" x2="49.618" y2="12.0024" width="0.254" layer="16"/>
+<wire x1="49.618" y1="12.0024" x2="46.99" y2="14.6304" width="0.254" layer="16"/>
 </signal>
 <signal name="D4_1">
@@
 <contactref element="U$1" pad="D4"/>
 <wire x1="13.486" y1="18.646" x2="15.622" y2="16.51" width="0.254" layer="16"/>
-<wire x1="26.5176" y1="10.5664" x2="33.528" y2="10.5664" width="0.254" layer="16"/>
+<wire x1="26.5176" y1="10.5664" x2="38.862" y2="10.5664" width="0.254" layer="16"/>
 <wire x1="15.622" y1="16.51" x2="20.574" y2="16.51" width="0.254" layer="16"/>
 <wire x1="20.574" y1="16.51" x2="26.5176" y2="10.5664" width="0.254" layer="16"/>
@@
 </board>
 </drawing>
+<compatibility>
+<note version="8.2" severity="warning">
+Since Version 8.2, EAGLE supports online libraries. The ids
+of those online libraries will not be understood (or retained)
+with this version.
+</note>
+<note version="8.3" severity="warning">
+Since Version 8.3, EAGLE supports URNs for individual library
+assets (packages, symbols, and devices). The URNs of those assets
+will not be understood (or retained) with this version.
+</note>
+<note version="8.3" severity="warning">
+Since Version 8.3, EAGLE supports the association of 3D packages
+with devices in libraries, schematics, and board files. Those 3D
+packages will not be understood (or retained) with this version.
+</note>
+</compatibility>
 </eagle>
